Commit message: dsadas

File: description/lidar.xacro (robot description, xacro)
@@ -20,8 +20,8 @@
         </collision>
         <inertial>
-            <mass value="0.1" />
-            <inertia ixx="${(1/12) * 0.1 * (3*.05*.05 + 0.04*0.04)}" ixy="0.0" ixz="0.0"
-                    iyy="${(1/12) * 0.1 * (3*.05*.05 + 0.04*0.04)}" iyz="0.0"
-                    izz="${(1/2) * 0.1 * (.05*.05)}" />
+            <mass value="0.01" />
+            <inertia ixx="0.00005" ixy="0.0" ixz="0.0"
+                    iyy="0.00005" iyz="0.0"
+                    izz="0.00005" />
             <origin xyz = "0 0 0" rpy = "0 0 0"/>
         </inertial>

File: description/robot.urdf.xacro (robot description, xacro)
@@ -1,7 +1,12 @@
 <?xml version="1.0"?>
 <robot xmlns:xacro="http://www.ros.org/wiki/xacro"  name="robot_bob">
-    <xacro:include filename="robot_core.xacro"/>
-    <!-- <xacro:include filename="gazebo_control.xacro"/> -->
-    <xacro:include filename="ros2_control.xacro"/>
+    <xacro:arg name="use_ros2_control" default="true"/>
+    <xacro:include filename="robot_core.xacro" />
+    <xacro:if value="$(arg use_ros2_control)">
+        <xacro:include filename="ros2_control.xacro" />
+    </xacro:if>
+    <xacro:unless value="$(arg use_ros2_control)">
+        <xacro:include filename="gazebo_control.xacro" />
+    </xacro:unless>
     <xacro:include filename="lidar.xacro"/>
     <xacro:include filename="camera.xacro"/>

File: description/robot_core copy.xacro (robot description, xacro)
@@ -20,5 +20,14 @@
 <!-- Base Link -->
   <link name="base_link">
+    <visual>
+      <origin xyz="0 0 0"/>
+      <geometry>
+        <box size="0.1 0.1 0.1" />
+      </geometry>
+    </visual>
   </link>
+  <gazebo reference="base_link">
+    <material>Gazebo/Red</material>
+  </gazebo>
 <!-- Chassis -->
     <joint name = "chassis_joint" type="fixed">
@@ -43,8 +52,8 @@
         <inertial>
             <mass value="1.0" />
-            <inertia ixx="0.00005" ixy="0.0" ixz="0.0"
-                    iyy="0.00005" iyz="0.0"
-                    izz="0.00005" />
-            <origin xyz = "0.15 0 0.075" rpy = "0 0 0"/>
+            <inertia ixx="${(1/12) * 1.0 * (0.3 *0.3 +0.15*0.15)}" ixy="0.0" ixz="0.0"
+                    iyy="${(1/12) * 1.0 * (0.3 *0.3 +0.15*0.15)}" iyz="0.0"
+                    izz="${(1/12) * 1.0 * (0.3 *0.3 +0.3 *0.3 )}" />
+            <origin xyz = "0.15 0 0.75" rpy = "0 0 0"/>
         </inertial>
     </link>
@@ -131,8 +140,8 @@
         </collision>
         <inertial>
-            <mass value="0.5" />
-            <inertia ixx="0.00005" ixy="0.0" ixz="0.0"
-                    iyy="0.00005" iyz="0.0"
-                    izz="0.00005" />
+            <mass value="1" />
+            <inertia ixx="${(2/5) * 0.1 * (0.05*0.05)}" ixy="0.0" ixz="0.0"
+                    iyy="${(2/5) * 0.1 * (0.05*0.05)}" iyz="0.0"
+                    izz="${(2/5) * 0.1 * (0.05*0.05)}" />
             <origin xyz = "0 0 0" rpy = "0 0 0"/>
         </inertial>
